File: SNSP-CPU-01/SNSP-CPU-01.kicad_pcb (KiCad board)
At the start: 2 copper layers, 215.8 x 159 mm, 400 parts, among them J1 Jack-DC, J3 Conn_02x06_Odd_Even, J4 CONTROLLER 1, J5 CONTROLLER 2, P1 CASSETTE, P2 JST 11FE-BT-VK-N, P3 Conn_01x02_Pin, P7 JST 11FE-BT-VK-N, Q10 C2412K, Q11 C2412K, Q12 C2412K, Q13 C2412K, Q14 C2412K, Q15 C2412K, Q16 C2412K, Q17 C2412K, Q18 2SC5658, Q3 C2412K, Q4 C2412K, Q5 C2412K, Q6 C2412K, Q7 C2412K, Q8 C2412K, Q9 C2412K, SW1 KB, SW2 Old, T1 L_Coupled, U1 CPU, U10 LM324, U11 LM809, U12 L7805, U13 S-SMP, U14 S-DSP, U15 MS62256CL-10FC, U16 MS62256CL-10FC, U17 uPD6376, U18 S-CLK, U2 PPU1, U3 PPU2, U4 MS62256CL-10FC, U5 MS62256CL-10FC, U6 WRAM, U7 S-ENC, U8 CIC, X1 17.734MHz, X2 24.576MHz

Commit message: Fixes the LR CLK issue
Parts:
- U17: value uPD6376 -> UPD6376
Connections:
- net //PARD renamed /~{PARD}
- net //PAWR renamed /~{PAWR}
- C73 pad 1: Net-(U14-LRCK) -> Net-(U17-L.REF)
- U17 pad 10: Net-(U14-LRCK) -> Net-(U17-L.REF)
- U17 pad 13: unconnected-(U17-LRCK/WDCK-Pad13) -> Net-(U14-LRCK)
- U17 pad 9: Net-(U14-LRCK) -> Net-(U17-L.REF)
Routing:
- net Net-(U17-L.REF): track 0.00 -> 11.8 mm
- net Net-(U14-LRCK): track 59.6 -> 54.9 mm, vias 2 -> 4
- net Net-(U13-CPUA13): track 37.9 -> 36.7 mm
- net Net-(U13-CPUA12): track 34.9 -> 33.8 mm
- net /RESOUT1: track 305.5 -> 304.5 mm
- net Net-(U13-CPUA14): track 39.8 -> 38.9 mm
- net /PA0: track 324.7 -> 324.0 mm
- net Net-(U13-CPUA15): track 42.5 -> 41.8 mm
- net Net-(U17-R.OUT): track 72.1 -> 72.8 mm
